Commit message: images of objects collected for detector training

File: simulation/models/apple/apple.urdf (robot description, URDF)
Before this commit: robot apple.urdf, 1 links, 0 joints
Links:
- link baseLink: geometry collision box size=0.05 0.05 0.05; visual mesh filename=apple.stl scale=0.0001 .0001 .0001

File: simulation/models/banana/banana.urdf (robot description, URDF)
Before this commit: robot banana.urdf, 1 links, 0 joints
Links:
- link baseLink: geometry collision box size=0.1 0.05 0.05; visual mesh filename=banana.stl scale=0.0005 .0005 .0005

File: simulation/models/milk/milk.urdf (robot description, URDF)
Before this commit: robot milk.urdf, 1 links, 0 joints
Links:
- link baseLink: geometry collision cylinder length=0.3 radius=0.2; visual mesh filename=milk.stl scale=.5 .5 .5

File: simulation/models/orange/orange.urdf (robot description, URDF)
Before this commit: robot orange.urdf, 1 links, 0 joints
Links:
- link baseLink: geometry collision box size=0.05 0.05 0.05; visual mesh filename=orange.stl scale=0.0005 .0005 .0005
