Commit message: integrated perception with action

File: simulation/models/container/container.urdf (robot description, URDF)
Before this commit: robot container.urdf, 1 links, 0 joints
Links:
- link baseLink: geometry collision box size=0.07 0.05 0.02; visual mesh filename=container.stl scale=1 1 1
