Commit message: confident bounding box and name implemented

File: simulation/models/bottle/bottle.urdf (robot description, URDF)
Before this commit: robot bottle.urdf, 1 links, 0 joints
Links:
- link baseLink: geometry collision box size=0.07 0.05 0.02; visual mesh filename=bottle.stl scale=0.001 .001 .001

File: simulation/models/coke/coke.urdf (robot description, URDF)
Before this commit: robot coke.urdf, 1 links, 0 joints
Links:
- link baseLink: geometry collision box size=0.07 0.05 0.02; visual mesh filename=coke.stl scale=0.001 .001 .001

File: simulation/models/lysol/lysol.urdf (robot description, URDF)
Before this commit: robot lysol.urdf, 1 links, 0 joints
Links:
- link baseLink: geometry collision box size=0.07 0.05 0.2; visual mesh filename=lysol.stl scale=1 1 1

Commit message: full box arrangement implemented

File: simulation/models/bottle/bottle.urdf (robot description, URDF)
Before this commit: robot bottle.urdf, 1 links, 0 joints
Links:
- link baseLink: geometry collision box size=0.02 0.05 0.02; visual mesh filename=bottle.stl scale=0.001 .001 .001

File: simulation/models/coke/coke.urdf (robot description, URDF)
Before this commit: robot coke.urdf, 1 links, 0 joints
Links:
- link baseLink: geometry collision box size=0.02 0.05 0.02; visual mesh filename=coke2.stl scale=1 1 1

File: simulation/models/lysol/lysol.urdf (robot description, URDF)
Before this commit: robot lysol.urdf, 1 links, 0 joints
Links:
- link baseLink: geometry collision box size=0.07 0.05 0.02; visual mesh filename=lysol.stl scale=1 1 1

File: simulation/models/pepsi/pepsi.urdf (robot description, URDF)
Before this commit: robot pepsi.urdf, 1 links, 0 joints
Links:
- link baseLink: geometry collision box size=0.02 0.02 0.02; visual mesh filename=pepsi.stl scale=0.001 .001 .001
