Commit message: implemented put-on and put-in-clutter

File: simulation/models/lipton/lipton.urdf (robot description, URDF)
Before this commit: robot lipton.urdf, 1 links, 0 joints
Links:
- link baseLink: geometry collision box size=0.02 0.02 0.02; visual mesh filename=lipton.stl scale=1 1 1

File: simulation/models/pepsi/pepsi.urdf (robot description, URDF)
Before this commit: robot pepsi.urdf, 1 links, 0 joints
Links:
- link baseLink: geometry collision box size=0.02 0.02 0.02; visual mesh filename=pepsi.stl scale=0.001 0.001 0.001
