Commit message: made some improvements to space constraint

File: simulation/models/ambrosia/ambrosia.urdf (robot description, URDF)
Before this commit: robot ambrosia.urdf, 1 links, 0 joints
Links:
- link baseLink: geometry collision box size=0.005 0.005 0.005; visual mesh filename=ambrosia.stl scale=1 1 1

File: simulation/models/apple/apple.urdf (robot description, URDF)
Before this commit: robot apple.urdf, 1 links, 0 joints
Links:
- link baseLink: geometry collision box size=0.005 0.005 0.005; visual mesh filename=apple.stl scale=0.0001 .0001 .0001

File: simulation/models/banana/banana.urdf (robot description, URDF)
Before this commit: robot banana.urdf, 1 links, 0 joints
Links:
- link baseLink: geometry collision box size=0.005 0.005 0.005; visual mesh filename=banana.stl scale=0.0005 .0005 .0005

File: simulation/models/bottle/bottle.urdf (robot description, URDF)
Before this commit: robot bottle.urdf, 1 links, 0 joints
Links:
- link baseLink: geometry collision box size=0.005 0.005 0.005; visual mesh filename=bottle.stl scale=0.001 .001 .001

File: simulation/models/cereal/cereal.urdf (robot description, URDF)
Before this commit: robot cereal.urdf, 1 links, 0 joints
Links:
- link baseLink: geometry collision box size=0.005 0.005 0.005; visual mesh filename=cereal.stl scale=0.001 .001 .001

File: simulation/models/coke/coke.urdf (robot description, URDF)
Before this commit: robot coke.urdf, 1 links, 0 joints
Links:
- link baseLink: geometry collision box size=0.005 0.005 0.005; visual mesh filename=coke2.stl scale=1 1 1

File: simulation/models/container/container.urdf (robot description, URDF)
Before this commit: robot container.urdf, 1 links, 0 joints
Links:
- link baseLink: geometry collision box size=0.005 0.005 0.005; visual mesh filename=container.stl scale=1 1 1

File: simulation/models/lipton/lipton.urdf (robot description, URDF)
Before this commit: robot lipton.urdf, 1 links, 0 joints
Links:
- link baseLink: geometry collision box size=0.005 0.005 0.005; visual mesh filename=lipton.stl scale=1 1 1

File: simulation/models/lysol/lysol.urdf (robot description, URDF)
Before this commit: robot lysol.urdf, 1 links, 0 joints
Links:
- link baseLink: geometry collision box size=0.005 0.005 0.005; visual mesh filename=lysol.stl scale=1 1 1

File: simulation/models/milk/milk.urdf (robot description, URDF)
Before this commit: robot milk.urdf, 1 links, 0 joints
Links:
- link baseLink: geometry collision box size=0.005 0.005 0.005; visual mesh filename=milk.stl scale=.5 .5 .5

File: simulation/models/nutella/nutella.urdf (robot description, URDF)
Before this commit: robot nutella.urdf, 1 links, 0 joints
Links:
- link baseLink: geometry collision box size=0.005 0.005 0.005; visual mesh filename=nutella.stl scale=1 1 1

File: simulation/models/orange/orange.urdf (robot description, URDF)
Before this commit: robot orange.urdf, 1 links, 0 joints
Links:
- link baseLink: geometry collision box size=0.005 0.005 0.005; visual mesh filename=orange.stl scale=0.0005 .0005 .0005

File: simulation/models/oreo/oreo.urdf (robot description, URDF)
Before this commit: robot oreo.urdf, 1 links, 0 joints
Links:
- link baseLink: geometry collision box size=0.005 0.005 0.005; visual mesh filename=oreo.stl scale=1 1 1

File: simulation/models/pepsi/pepsi.urdf (robot description, URDF)
Before this commit: robot pepsi.urdf, 1 links, 0 joints
Links:
- link baseLink: geometry collision box size=0.005 0.005 0.005; visual mesh filename=pepsi.stl scale=0.001 0.001 0.001
